File: Hardware/Eagle/C128_Ultimate.sch (EAGLE design)
At the start: 3 parts, among them IC1 0RB_COMMODORE_EXPANSION_PORT_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, X4 TSW-122-07-G-Q

Commit message: Update Hardware/Eagle/C128_Ultimate.sch
Properly moved reset button to bottom side
Connections:
- net !RES: now also S1.1; no longer S1.2
- net GND: now also S1.2; no longer S1.1
Changed lines of the file:
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@@
 <?xml version="1.0" encoding="utf-8"?>
 <!DOCTYPE eagle SYSTEM "eagle.dtd">
-<eagle version="8.6.0">
+<eagle version="9.0.1">
 <drawing>
 <settings>
@@
 <wire x1="163.83" y1="153.67" x2="163.83" y2="151.13" width="0.1524" layer="91"/>
 <wire x1="163.83" y1="151.13" x2="167.64" y2="147.32" width="0.1524" layer="91"/>
-<pinref part="S1" gate="G$1" pin="1"/>
-<wire x1="154.94" y1="165.1" x2="154.94" y2="157.48" width="0.1524" layer="91"/>
-<wire x1="154.94" y1="157.48" x2="160.02" y2="157.48" width="0.1524" layer="91"/>
-<wire x1="160.02" y1="157.48" x2="163.83" y2="153.67" width="0.1524" layer="91"/>
 <wire x1="167.64" y1="147.32" x2="172.72" y2="147.32" width="0.1524" layer="91"/>
+<wire x1="163.83" y1="153.67" x2="163.83" y2="160.02" width="0.1524" layer="91"/>
+<wire x1="163.83" y1="160.02" x2="165.1" y2="160.02" width="0.1524" layer="91"/>
+<pinref part="S1" gate="G$1" pin="2"/>
+<wire x1="165.1" y1="160.02" x2="165.1" y2="165.1" width="0.1524" layer="91"/>
 </segment>
 <segment>
@@
 </segment>
 <segment>
-<pinref part="S1" gate="G$1" pin="2"/>
-<wire x1="165.1" y1="165.1" x2="132.08" y2="165.1" width="0.1524" layer="91"/>
-</segment>
-</net>
+<pinref part="S1" gate="G$1" pin="1"/>
+<wire x1="154.94" y1="165.1" x2="152.4" y2="165.1" width="0.1524" layer="91"/>
+<wire x1="152.4" y1="165.1" x2="152.4" y2="154.94" width="0.1524" layer="91"/>
+</segment>
+</net>

Commit message: Update Hardware/Eagle/C128_Ultimate.sch
Other:
- note added: "Cartridge Vertical to Horizontal adapter"
- note added: "Designer: Tomse"
Changed lines of the file:
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@@
 </classes>
 <parts>
-<part name="FRAME1" library="SparkFun-Aesthetics" library_urn="urn:adsk.eagle:library:507" deviceset="FRAME-A4L" device=""/>
+<part name="FRAME1" library="SparkFun-Aesthetics" library_urn="urn:adsk.eagle:library:507" deviceset="FRAME-A4L" device="">
+<attribute name="DESIGNER" value="Copyright (c) 2018 http://retro-commodore.eu"/>
+</part>
 <part name="GND2" library="supply1" library_urn="urn:adsk.eagle:library:371" deviceset="GND" device=""/>
 <part name="IC1" library="C64CartridgeEdgeConnector" deviceset="0RB_COMMODORE_EXPANSION_PORT_C64" device=""/>
@@
 <sheet>
 <plain>
+<text x="185.42" y="20.32" size="2.54" layer="94">Cartridge Vertical to Horizontal adapter</text>
+<text x="185.42" y="10.16" size="2.54" layer="94">Designer: Tomse</text>
 </plain>
 <instances>
-<instance part="FRAME1" gate="G$1" x="19.05" y="3.81"/>
+<instance part="FRAME1" gate="G$1" x="3.81" y="3.81" smashed="yes">
+<attribute name="SHEET" x="199.39" y="5.08" size="2.54" layer="94" font="vector"/>
+<attribute name="DESIGNER" x="185.366" y="15.24" size="2.54" layer="94" font="vector"/>
+<attribute name="CREVISION" x="238.73" y="4.98" size="2.54" layer="94" font="vector"/>
+</instance>
 <instance part="GND2" gate="1" x="166.37" y="153.67" rot="R90"/>
 <instance part="IC1" gate="G$7" x="58.42" y="116.84"/>
